File: vampire_pcb/kicad_project/vampire_pcb.kicad_sch (KiCad schematic)
At the start: 4 parts, among them J1 VAMPIRE_EDGE, J2 GND_PAD, J3 Conn_01x08, J4 Conn_01x08

Commit message: Update PCB
Parts:
- removed J4: Conn_01x08, Connector_JST:JST_PH_B8B-PH-K_1x08_P2.00mm_Vertical, symbol Connector_Generic:Conn_01x08
- renumbered J3 to J1, J1 to J2, J2 to J3
