File: gain_box/kicad_project/gain_box.kicad_pcb (KiCad board)
At the start: 2 copper layers, 167.5 x 101.5 mm, 76 parts, among them J1 Conn_01x02, J10 AVR-UPDI-6, J11 Conn_01x02, J2 Conn_01x02, J3 Conn_01x02, J4 Conn_01x02, J5 Conn_01x02, J6 Conn_01x02, J7 Conn_01x02, J8 Conn_01x02, J9 Conn_01x02, K1 G5V-1, K2 G5V-1, K3 G5V-1, K4 J107F1CS2012VDC.80, K5 J107F1CS2012VDC.80, Q1 AO3400A, Q2 AO3400A, Q3 AO3400A, T1 70042K, U1 NE5532, U10 140817141310, U2 NE5532, U3 NE5532, U4 LM7809, U5 LM7909, U6 LM7805_TO220, U7 ATtiny412-SS, U9 140817141310

Commit message: gain_box: preliminary amp section layout
Parts:
- removed RN1: 4x10K, Resistor_SMD:R_Array_Convex_4x1206
- added C10: 100n, Capacitor_THT:C_Disc_D3.8mm_W2.6mm_P2.50mm, F.Cu at (87.5, 114.5)
- added C11: 100n, Capacitor_THT:C_Disc_D3.8mm_W2.6mm_P2.50mm, F.Cu at (-49.7, 117.6)
- added C12: 100n, Capacitor_THT:C_Disc_D3.8mm_W2.6mm_P2.50mm, F.Cu at (-49.7, 121.8)
- added C13: 100n, Capacitor_THT:C_Disc_D3.8mm_W2.6mm_P2.50mm, F.Cu at (-44.1, 113.5)
- added C14: 100n, Capacitor_THT:C_Disc_D3.8mm_W2.6mm_P2.50mm, F.Cu at (-44.1, 117.6)
- added C15: 100n, Capacitor_THT:C_Disc_D3.8mm_W2.6mm_P2.50mm, F.Cu at (-44.1, 121.8)
- added C16: 100n, Capacitor_THT:C_Disc_D3.8mm_W2.6mm_P2.50mm, F.Cu at (-38.4, 113.5)
- added C17: 100n, Capacitor_THT:C_Disc_D3.8mm_W2.6mm_P2.50mm, F.Cu at (-38.5, 117.8)
- added C18: 100n, Capacitor_THT:C_Disc_D3.8mm_W2.6mm_P2.50mm, F.Cu at (-38.4, 121.8)
- added C19: 330n, Capacitor_THT:C_Disc_D7.5mm_W4.4mm_P5.00mm, F.Cu at (-49.3, 126.8)
- added C20: 2200u, Capacitor_THT:CP_Radial_D16.0mm_P7.50mm, F.Cu at (-142.6, 24.7)
- added C21: 2200u, Capacitor_THT:CP_Radial_D16.0mm_P7.50mm, F.Cu at (-142.6, 42.3)
- added C22: 2200u, Capacitor_THT:CP_Radial_D16.0mm_P7.50mm, F.Cu at (-142.6, 59.8)
- added C23: 2200u, Capacitor_THT:CP_Radial_D16.0mm_P7.50mm, F.Cu at (-142.6, 77.4)
- added C24: 10u, Capacitor_THT:CP_Radial_D5.0mm_P2.00mm, F.Cu at (-60.6, 42.6)
- added C25: 10u, Capacitor_THT:CP_Radial_D5.0mm_P2.00mm, F.Cu at (-60.6, 49.2)
- added C26: 10u, Capacitor_THT:CP_Radial_D5.0mm_P2.00mm, F.Cu at (-60.6, 55.7)
- added C27: 10u, Capacitor_THT:CP_Radial_D5.0mm_P2.00mm, F.Cu at (-60.6, 62.3)
- added C4: 10n, Capacitor_THT:C_Rect_L7.2mm_W2.5mm_P5.00mm_FKS2_FKP2_MKS2_MKP2, F.Cu at (90.0, 99.2)
- added C5: 10n, Capacitor_THT:C_Rect_L7.2mm_W2.5mm_P5.00mm_FKS2_FKP2_MKS2_MKP2, F.Cu at (-146.2, 105.6)
- added C6: 10n, Capacitor_THT:C_Rect_L7.2mm_W2.5mm_P5.00mm_FKS2_FKP2_MKS2_MKP2, F.Cu at (-146.2, 109.7)
- added C7: 3.3u, Capacitor_THT:C_Rect_L13.0mm_W6.0mm_P10.00mm_FKS3_FKP3_MKS4, F.Cu at (77.8, 109.5)
- added C8: 3.3u, Capacitor_THT:C_Rect_L13.0mm_W6.0mm_P10.00mm_FKS3_FKP3_MKS4, F.Cu at (-54.0, 50.7)
- added C9: 3.3u, Capacitor_THT:C_Rect_L13.0mm_W6.0mm_P10.00mm_FKS3_FKP3_MKS4, F.Cu at (-54.0, 58.2)
- added R25: 33k, Resistor_SMD:R_0805_2012Metric_Pad1.20x1.40mm_HandSolder, F.Cu at (-58.4, 124.7)
- added R26: 33k, Resistor_SMD:R_0805_2012Metric_Pad1.20x1.40mm_HandSolder, F.Cu at (-58.4, 127.6)
- added R27: 10k, Resistor_SMD:R_0805_2012Metric_Pad1.20x1.40mm_HandSolder, F.Cu at (-53.7, 112.9)
- added R28: 10k, Resistor_SMD:R_0805_2012Metric_Pad1.20x1.40mm_HandSolder, F.Cu at (-53.7, 115.8)
- added R29: 10k, Resistor_SMD:R_0805_2012Metric_Pad1.20x1.40mm_HandSolder, F.Cu at (-53.7, 118.8)
- added R30: 10k, Resistor_SMD:R_0805_2012Metric_Pad1.20x1.40mm_HandSolder, F.Cu at (-53.7, 121.7)
- added RV4: 300VAC, Varistor:RV_Disc_D9mm_W4.5mm_P5mm, F.Cu at (-145.3, 125.6)
- added TP1: TestPoint, TestPoint:TestPoint_Pad_D2.0mm, F.Cu at (-44.9, 75.2)
- added TP10: TestPoint, TestPoint:TestPoint_Pad_D2.0mm, F.Cu at (-40.8, 91.4)
- added TP11: TestPoint, TestPoint:TestPoint_Pad_D2.0mm, F.Cu at (-36.8, 75.2)
- added TP12: TestPoint, TestPoint:TestPoint_Pad_D2.0mm, F.Cu at (-36.8, 79.2)
- added TP13: TestPoint, TestPoint:TestPoint_Pad_D2.0mm, F.Cu at (-36.8, 83.3)
- added TP14: TestPoint, TestPoint:TestPoint_Pad_D2.0mm, F.Cu at (-36.8, 87.3)
- added TP2: TestPoint, TestPoint:TestPoint_Pad_D2.0mm, F.Cu at (-44.9, 79.2)
- added TP3: TestPoint, TestPoint:TestPoint_Pad_D2.0mm, F.Cu at (-44.9, 83.3)
- added TP4: TestPoint, TestPoint:TestPoint_Pad_D2.0mm, F.Cu at (-44.9, 87.3)
- added TP5: TestPoint, TestPoint:TestPoint_Pad_D2.0mm, F.Cu at (-44.9, 91.4)
- added TP6: TestPoint, TestPoint:TestPoint_Pad_D2.0mm, F.Cu at (-40.8, 75.2)
- added TP7: TestPoint, TestPoint:TestPoint_Pad_D2.0mm, F.Cu at (-40.8, 79.2)
- added TP8: TestPoint, TestPoint:TestPoint_Pad_D2.0mm, F.Cu at (-40.8, 83.3)
- added TP9: TestPoint, TestPoint:TestPoint_Pad_D2.0mm, F.Cu at (-40.8, 87.3)
- C1, C2, C3: footprint Capacitor_THT:C_Rect_L26.5mm_W10.5mm_P22.50mm_MKS4 -> Capacitor_THT:C_Rect_L7.2mm_W4.5mm_P5.00mm_FKS2_FKP2_MKS2_MKP2
- K1, K2: value G5V-1 -> J104D2C12VDC.36S
- K4: footprint gain_box:RELAY_SRD-05VDC-SL-C -> gain_box:RELAY_SRD-C
- K5: value J107F1CS2012VDC.80 -> J104D2C12VDC.36S
- R1, R10, R11, R12, R13, R14, R15, R2, R22, R23, R24, R3, R4, R5, R6, R7, R8, R9: footprint Resistor_THT:R_Axial_DIN0204_L3.6mm_D1.6mm_P7.62mm_Horizontal -> Resistor_THT:R_Axial_DIN0207_L6.3mm_D2.5mm_P7.62mm_Horizontal
- R20, R21: value 2.2k -> 10k
- U6: value LM7805_TO220 -> 78L05; footprint Package_TO_SOT_THT:TO-220-3_Vertical -> Package_TO_SOT_SMD:SOT-89-3
- moved K4 360.0 mm to (-120.9, 141.0)
- moved F1 357.8 mm to (-127.2, 113.7)
- moved RV2 343.8 mm to (-100.4, 121.4)
- moved RV3 343.8 mm to (-100.4, 127.8)
- moved U9 322.0 mm to (-146.4, 88.2)
- moved U10 320.3 mm to (-146.4, 94.9)
- moved U4 318.7 mm to (-144.8, 115.6)
- moved U5 318.7 mm to (-144.8, 121.6)
- moved K5 309.7 mm to (-80.6, 118.2)
- moved U6 292.1 mm to (-118.2, 123.7)
- moved J10 287.5 mm to (-137.0, 101.9)
- moved R11 287.2 mm to (-72.0, 49.0)
- moved R14 287.2 mm to (-72.0, 58.5)
- moved R15 287.2 mm to (-72.0, 61.6)
- moved R2 287.2 mm to (-72.0, 20.7)
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Connections:
- net AC_OK renamed AC_PULSE
- net AC_SENSE_1 renamed AC_SENSE
- net AC_SENSE_2 renamed AGND
- net Net-(J8-Pin_2) renamed TGO1
- net Net-(J9-Pin_2) renamed TGO2
- F1 pad 1: Net-(J11-Pin_3) -> Net-(J11-Pin_2)
- J11 pad 2: unconnected-(J11-Pin_2-Pad2) -> Net-(J11-Pin_2)
- U6 pad 1: +12V -> +5V
- U6 pad 3: +5V -> +12V
Routing:
- net AGND: track 0.00 -> 76.4 mm
- net Net-(U1A--): track 0.00 -> 32.1 mm
- net Net-(C7-Pad1): track 0.00 -> 20.5 mm
- net Net-(U1A-+): track 0.00 -> 16.8 mm
- net AV+: track 0.00 -> 14.6 mm
- net Net-(C7-Pad2): track 0.00 -> 13.5 mm
- net OUT_FL: track 0.00 -> 10.0 mm
- net IN_FL: track 0.00 -> 7.30 mm
- net AV-: track 0.00 -> 6.50 mm
- net Net-(C1-Pad2): track 0.00 -> 3.69 mm
Other:
- board outline removed

Commit message: gain_box: first audio PSU layout
Parts:
- moved C6 320.5 mm to (168.9, 51.2), turned to -90 degrees
- moved C5 316.5 mm to (169.0, 77.2), turned to -90 degrees
- moved RV3 293.8 mm to (186.2, 63.2), turned to 180 degrees
- moved U2 290.3 mm to (172.2, 84.2), turned to 90 degrees
- moved RV2 288.4 mm to (186.3, 89.2), turned to 180 degrees
- moved U3 282.3 mm to (172.1, 58.2), turned to 90 degrees
- moved R11 265.2 mm to (190.8, 84.5), turned to 90 degrees
- moved C3 264.1 mm to (160.2, 51.7)
- moved R12 262.6 mm to (190.7, 58.5), turned to 90 degrees
- moved R24 260.0 mm to (187.2, 50.8), turned to -90 degrees
- moved R23 259.4 mm to (187.2, 76.9), turned to -90 degrees
- moved C2 256.9 mm to (160.2, 77.7)
- moved K4 249.1 mm to (109.1, 45.4), turned to 180 degrees
- moved R2 246.1 mm to (166.3, 82.2), turned to 180 degrees
- moved C12 243.2 mm to (183.7, 53.4), turned to 90 degrees
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Connections:
- F1 pad 1: Net-(J11-Pin_2) -> Net-(J11-Pin_1)
- J11 pad 1: AC_N -> Net-(J11-Pin_1)
- J11 pad 2: Net-(J11-Pin_2) -> AC_N
- T1 pad 3: AC_N -> AC_L_SW
- T1 pad 6: AC_L_SW -> AC_N
Routing:
- net AGND: track 76.4 -> 383.7 mm
- net AC_L: track 0.00 -> 126.0 mm
- net AC_N: track 0.00 -> 87.7 mm
- net AV+: track 14.6 -> 69.7 mm
- net Net-(D12-A): track 0.00 -> 43.4 mm
- net Net-(D11-K): track 0.00 -> 39.2 mm
- net AV-: track 6.50 -> 45.3 mm
- net Net-(T1-Pad4): track 0.00 -> 35.6 mm
- net Net-(U3A--): track 0.00 -> 32.2 mm
- net Net-(U2A--): track 0.00 -> 32.2 mm
- net Net-(D7-K): track 0.00 -> 25.9 mm
- net Net-(D10-A): track 0.00 -> 25.8 mm
- net Net-(C8-Pad1): track 0.00 -> 20.1 mm
- net Net-(C9-Pad1): track 0.00 -> 20.1 mm
- net Net-(C9-Pad2): track 0.00 -> 12.9 mm
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- added copper zone on F.Cu, net AGND
Other:
- board outline added: 160 x 90 mm
- board text added: "AGND"
- board text added: "AV+"
- board text added: "AV-"
- board text added: "C"
- board text added: "GAIN"
- board text added: "IN"
- board text added: "L"
- board text added: "OUT"
- board text added: "R"

Commit message: gain_box new PSU position
Parts:
- removed the K1 at (132.9, 107.0)
- moved J7 213.3 mm to (139.2, 115.7)
- moved J8 202.9 mm to (130.0, 115.8)
- moved U7 202.5 mm to (132.5, 107.0)
- moved U10 199.7 mm to (141.5, 111.5), turned to 90 degrees
- moved C13 196.7 mm to (124.2, 103.7), turned to -90 degrees
- moved J9 193.0 mm to (121.0, 115.8)
- moved R19 192.4 mm to (138.0, 111.8)
- moved D1 189.7 mm to (125.2, 52.2)
- moved D2 189.2 mm to (125.3, 97.5)
- moved J10 178.1 mm to (138.2, 100.8), turned to 90 degrees
- moved TP4 174.0 mm to (129.9, 100.7)
- moved TP5 168.3 mm to (124.7, 100.8)
- moved U6 165.2 mm to (119.5, 104.9), turned to -90 degrees
- moved TP6 164.8 mm to (120.2, 111.0)
- moved U9 158.3 mm to (100.2, 100.3), turned to -90 degrees
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- renumbered K2 to K1
Connections:
- K1 pad 12: OUT_CEN -> OUT_FL
- K3 pad 21: AGND -> unconnected-(K3-Pad21)
- K3 pad 22: OUT_FR -> unconnected-(K3-Pad22)
- T1 pad 11: AC_SENSE -> Net-(D10-K)
- T1 pad 14: Net-(D10-K) -> AC_SENSE
- T1 pad 3: AC_L_SW -> AC_N
- T1 pad 6: AC_N -> AC_L_SW
Routing:
- net AV-: track 45.3 -> 221.6 mm, vias 0 -> 4
- net +12V: track 0.00 -> 142.2 mm
- net AV+: track 69.7 -> 206.6 mm
- net AGND: track 383.7 -> 515.1 mm
- net AC_SENSE: track 3.74 -> 68.2 mm
- net AC_L: track 126.0 -> 68.1 mm
- net OUT_FL: track 5.04 -> 37.2 mm
- net UNMUTE_G: track 0.00 -> 30.4 mm
- net Net-(D10-K): track 3.74 -> 28.9 mm
- net OUT_FR: track 5.04 -> 24.5 mm, vias 0 -> 1
- net OUT_CEN: track 5.04 -> 23.3 mm, vias 0 -> 2
- net Net-(D10-A): track 25.8 -> 37.9 mm
- net Net-(D7-K): track 25.9 -> 35.1 mm
- net Net-(D11-K): track 39.2 -> 30.4 mm
- net Net-(D12-A): track 43.4 -> 35.5 mm
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Other:
- board size 160 x 90 mm -> 160 x 84.2 mm
- board text added: "12V"
- board text added: "5V"
- board text added: "AC_PLS"
- board text added: "GND"
